File: butterfly.kicad_pcb (KiCad board)
At the start: 2 copper layers, 193.5 x 116.6 mm, 64 parts, among them J1 USB_C_Receptacle_USB2.0, SW1 BOOT, SW2 RESET, U2 USBLC6-2SC6

Commit message: before ground-hexing
Parts:
- added G*** (x2): LOGO, LOGO, B.Cu at (93.0, 103.1)
- turned D2 to -90 degrees
Routing:
- net Net-(D2-A-Pad1): track 112.5 -> 114.1 mm
- net Net-(D2-A-Pad2): track 95.4 -> 94.3 mm
